File: my-keyboard/my-keyboard.kicad_sch (KiCad schematic)
At the start: 26 parts, among them J1 USB_C_Receptacle_USB2.0, J2 ISP, SW1 RESET, U1 ATmega32U4-A, U2 AMS1117-3.3, Y1 8MHz

Commit message: Update PCB layout
Connections:
- net COL_3: now reaches U1.1 (PE6)
- net COL_5: now reaches U1.12 (PB7)
- net COL_6: now reaches U1.18 (PD0)
- net COL_7: now reaches U1.19 (PD1)
- net COL_8: now reaches U1.20 (PD2)
- net COL_9: now reaches U1.21 (PD3)
- net COL_10: now reaches U1.22 (PD5)
- net COL_11: now reaches U1.26 (PD6)
- net COL_12: now reaches U1.27 (PD7)
- net COL_13: now reaches U1.28 (PB4)
- net COL_14: now reaches U1.29 (PB5)
- net COL_0: now reaches U1.31 (PC6)
- net COL_1: now reaches U1.32 (PC7)
- net COL_2: now reaches U1.36 (PF7)
- net ROW_0: now reaches U1.37 (PF6)
- net ROW_1: now reaches U1.38 (PF5)
- net ROW_2: now reaches U1.39 (PF4)
- net ROW_3: now reaches U1.40 (PF1)
- net ROW_4: now reaches U1.41 (PF0)
- net COL_4: now reaches U1.8 (PB0)
Other:
- title: (none) -> My Keyboard
